File: Resources_PCB_Schematics/KiCadMotherBoard/KiCadMotherBoard_oneController.kicad_sch (KiCad schematic)
At the start: 20 parts, among them J1 Conn_01x04_Male, J10 Conn_01x04_Male, J11 Conn_01x04_Male, J12 Conn_01x04_Male, J13 SDA_SCL_BRIDGE, J14 SDA_SCL_BRIDGE, J2 Conn_01x04_Male, J3 Conn_01x04_Male, J4 Conn_01x04_Male, J5 Conn_01x04_Male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

Commit message: implementing
Parts:
- added J15, J16: SDA_SCL_BRIDGE, Connector_JST:JST_XH_B2B-XH-AM_1x02_P2.50mm_Vertical, symbol Connector:Conn_01x02_Male
- added U2: LED_CONTROLLER, ESP32_devkit_v1:esp32_devkit_v1_doit, symbol ESP32_devkit_v1:ESP32_DevKit_V1_DOIT
Connections:
- net +5V: now also U2.15 (VIN)
- net GND: now also U3.7 (REXT), U2.14 (GND); no longer U3.6 (VSS)
- net LED_P12: now also J11.1 (Pin_1), U2.12 (IO12); no longer J2.1 (Pin_1), U1.12 (IO12)
- net LED_P13: now also J12.1 (Pin_1), U2.13 (IO13); no longer J1.1 (Pin_1), U1.13 (IO13)
- net LED_P14: now also J6.1 (Pin_1), U2.11 (IO14); no longer J3.1 (Pin_1), U1.11 (IO14)
- net LED_P19: now also J8.1 (Pin_1), U2.25 (IO19); no longer J7.1 (Pin_1), U1.25 (IO19)
- net LED_P23: now also J7.1 (Pin_1), U2.30 (IO23); no longer J9.1 (Pin_1), U1.30 (IO23)
- net LED_P25: now also J3.1 (Pin_1), U2.8 (IO25); no longer J10.1 (Pin_1), U1.8 (IO25)
- net LED_P26: now also J4.1 (Pin_1), U2.9 (IO26); no longer J5.1 (Pin_1), U1.9 (IO26)
- net LED_P27: now also J5.1 (Pin_1), U2.10 (IO27); no longer J4.1 (Pin_1), U1.10 (IO27)
- net LED_P32: now also J1.1 (Pin_1), U2.6 (IO32); no longer J12.1 (Pin_1), U1.6 (IO32)
- net LED_P33: now also J2.1 (Pin_1), U2.7 (IO33); no longer J11.1 (Pin_1), U1.7 (IO33)
- net SCL: now also J15.2 (Pin_2), J16.2 (Pin_2), U2.29 (IO22)
- net SDA: now also J15.1 (Pin_1), J16.1 (Pin_1), U2.26 (IO21)
- net TOUCH1: now also J9.4 (Pin_4); no longer J3.4 (Pin_4)
- net TOUCH10: now also J3.4 (Pin_4); no longer J12.4 (Pin_4)
- net TOUCH11: now also J2.4 (Pin_4); no longer J11.4 (Pin_4)
- net TOUCH12: now also J1.4 (Pin_4); no longer J10.4 (Pin_4)
- net TOUCH2: now also J10.4 (Pin_4); no longer J2.4 (Pin_4)
- net TOUCH3: now also J11.4 (Pin_4); no longer J1.4 (Pin_4)
- net TOUCH4: now also J12.4 (Pin_4); no longer J4.4 (Pin_4)
- net TOUCH5: now also J8.4 (Pin_4); no longer J5.4 (Pin_4)
- net TOUCH6: now also J7.4 (Pin_4); no longer J6.4 (Pin_4)
- net TOUCH7: now also J6.4 (Pin_4); no longer J7.4 (Pin_4)
- net TOUCH8: now also J5.4 (Pin_4); no longer J8.4 (Pin_4)
- net TOUCH9: now also J4.4 (Pin_4); no longer J9.4 (Pin_4)
- net MAIN_CONTROLLER_3V3: now reaches U1.16 (3V3)
- net LED_P3: no longer names the net of U1.27 (RXD0/IO3)
- net LED_P3: no longer J8.1 (Pin_1)
- net LED_P4: no longer names the net of U1.20 (IO4)
- net LED_P4: no longer J6.1 (Pin_1)
- new net LED_P18: J9.1 (Pin_1), U2.24 (IO18)
- new net LED_P5: J10.1 (Pin_1), U2.23 (IO5)
Other:
- moved on the sheet: J1, J10, J11, J12, J2, J3, J4, J5, J6, J7, J8, J9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
